File: ACIA.kicad_sch (KiCad schematic)
At the start: 17 parts, among them J11 TTL SERIAL CONSOLE, J12 TTL CONSOLE PWR, P17 1.8432 MHz CLK, P18 SERIAL, U49 MAX232

Commit message: initial commit
Parts:
- gave numbers to parts that had none: 1
Connections:
- net CTS_TTL: now also U49.9 (R2OUT)
- net RXD_TTL: no longer U49.9 (R2OUT)
Other:
- title: 6809PC -> 6502PC
- moved on the sheet: C65, J12
