File: Decoder.kicad_sch (KiCad schematic)
At the start: 5 parts, among them U1 74LS04, U21 74LS00, U23 74LS688, U24 74LS138, U7 74LS32

Commit message: initial commit
Other:
- title: 6809PC -> 6502PC
