File: ECBbus.kicad_sch (KiCad schematic)
At the start: 12 parts, among them J1 IRQ Selection, J10 Bus_ISA_8bit, J13 IRQ Selection, J14 Bus_ISA_8bit, J2 IRQ Selection, J3 Bus_ISA_8bit, J4 Bus_ISA_8bit, J5 IRQ Selection, J6 Bus_ISA_8bit, J7 IRQ Selection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

Commit message: initial commit
Other:
- title: 6809PC -> 6502PC
Changed lines of the file:
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@@
 (kicad_sch
-	(version 20231120)
+	(version 20250114)
 	(generator "eeschema")
-	(generator_version "8.0")
+	(generator_version "9.0")
 	(paper "USLedger")
 	(title_block
-		(title "6809PC")
-		(date "2025-06-20")
-		(rev "004")
-		(comment 1 "https://github.com/danwerner21/6809PC")
+		(title "6502PC")
+		(date "2025-10-05")
+		(rev "001")
+		(comment 1 "https://github.com/danwerner21/6502PC")
 		(comment 2 "Based on work by Andrew Lynch and John Coffman")
 	)
