File: IO.kicad_sch (KiCad schematic)
At the start: 15 parts, among them P13 14.31818 MHz CLK, U15 74LS08, U16 74LS32, U18 74LS06, U21 74LS00, U25 74LS245, U26 74LS245, U27 74LS245, U28 74LS245, U7 74LS32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

Commit message: initial commit
Other:
- title: 6809PC -> 6502PC
Changed lines of the file:
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@@
 (kicad_sch
-	(version 20231120)
+	(version 20250114)
 	(generator "eeschema")
-	(generator_version "8.0")
+	(generator_version "9.0")
 	(paper "B")
 	(title_block
-		(title "6809PC")
-		(date "2025-06-20")
-		(rev "004")
-		(comment 1 "https://github.com/danwerner21/6809PC")
+		(title "6502PC")
+		(date "2025-10-05")
+		(rev "001")
+		(comment 1 "https://github.com/danwerner21/6502PC")
 		(comment 2 "Based on work by Andrew Lynch and John Coffman")
 	)
+	(text "1"
+		(exclude_from_sim no)
+		(at 81.534 91.186 0)
+		(effects
+			(font
+				(size 1.27 1.27)
+			)
+		)
+	)
+	(text "Read from bus, Low  . . .  write to bus high.\n"
+		(exclude_from_sim no)
+		(at 143.51 89.154 0)
+		(effects
+			(font
+				(size 1.27 1.27)
+			)
+		)
+	)
 	(junction
 		(at 46.99 144.78)
@@
 		)
 	)
-	(text "1"
-		(exclude_from_sim no)
-		(at 81.534 91.186 0)
-		(effects
-			(font
-				(size 1.27 1.27)
-			)
-		)
-	)
-	(text "Read from bus, Low  . . .  write to bus high.\n"
-		(exclude_from_sim no)
-		(at 143.51 89.154 0)
-		(effects
-			(font
-				(size 1.27 1.27)
-			)
-		)
-	)
 	(label "GND"
 		(at 149.86 83.82 0)
-		(fields_autoplaced yes)
 		(effects
 			(font
@@
 	(label "VCC"
 		(at 306.07 25.4 0)
-		(fields_autoplaced yes)
 		(effects
 			(font
@@
 					(unit 1)
 				)
+			)
+		)
+	)
+	(symbol
+		(lib_id "power:GND")
+		(at 148.59 83.82 0)
+		(unit 1)
+		(exclude_from_sim no)
+		(in_bom yes)
+		(on_board yes)
+		(dnp no)
+		(property "Reference" "#PWR0178"
+			(at 148.59 83.82 0)
+			(effects
+				(font
+					(size 0.762 0.762)
+				)
+				(hide yes)
+			)
+		)
+		(property "Value" "GND"
+			(at 148.59 85.598 0)
+			(effects
+				(font
+					(size 0.762 0.762)
+				)
+				(hide yes)
+			)
+		)
+		(property "Footprint" ""
+			(at 148.59 83.82 0)
+			(effects
+				(font
+					(size 1.27 1.27)
+				)
+				(hide yes)
+			)
+		)
+		(property "Datasheet" ""
+			(at 148.59 83.82 0)
+			(effects
+				(font
+					(size 1.27 1.27)
+				)
+				(hide yes)
+			)
+		)
+		(property "Description" "Power symbol creates a global label with name \"GND\" , ground"
+			(at 148.59 83.82 0)
+			(effects
+				(font
+					(size 1.27 1.27)
+				)
+				(hide yes)
+			)
+		)
+		(pin "1"
+		)
+		(instances
+			(project "6502PC-6U"
+				(path "/d94f9d60-5ece-4752-b49c-b0d1c95f35bc/00000000-0000-0000-0000-0000526d5517"
+					(reference "#PWR0178")
+					(unit 1)
+				)
