File: MMU-4.kicad_sch (KiCad schematic)
At the start: 16 parts, among them U1 74LS04, U10 74LS32, U15 74LS08, U22 74LS74, U35 74LS174, U36 74LS244, U37 74LS157, U38 74LS374, U39 74LS244, U40 SRAM-32K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

Commit message: initial commit
Parts:
- removed unit 2 of U15
- removed unit 3 of U15
Connections:
- net BUSAK is gone; now on net GND: U43.15 (OE), U44.15 (OE), U45.19 (OEb), U46.1 (OEa), U46.19 (OEb)
- net /MMU-ENB-WR: no longer U42.13 (O2)
- net /MMU-MAP-RD: no longer U15.1
- net /MMU-MAP-WR: no longer U40.27 (~{WE})
- net /MMU-TASK-SETUP-WR: no longer U42.14 (O1)
- net /MMU-TASK-WR: no longer U42.15 (O0)
- net /RESET: now also U22.13 (~{R}), U35.1 (~{Mr})
- net /IOSEL-0EFD0: no longer U1.3, U41.19 (CE)
- net /MMU-TASK-RD renamed /MMU-TASK-RD
- net CPU_Q: no longer names the net of U45.4 (I1a)
- net Q: no longer names the net of U45.16 (O1a)
- new net /MMU-ENB-WR: U42.13 (O2)
- new net /MMU-MAP-RD: U15.1
- new net /MMU-MAP-RW: U1.3, U41.19 (CE)
- new net /MMU-MAP-WR: U40.27 (~{WE})
- new net /MMU-TASK-SETUP-WR: U42.14 (O1)
- new net /MMU-TASK-WR: U42.15 (O0)
- no-connect marks 14 -> 15
Other:
- note removed: "ECB bus signal"
- note removed: "rev. 011 -- change from /MMU-MAP-RW to MMU-ENABLE"
- title: 6809PC -> 6502PC
