File: Power.kicad_sch (KiCad schematic)
At the start: 88 parts, among them P10 CONN_1, P11 CONN_10X2, P12 POWER_SW, P2 CONN_1, P21 CONN_1, P22 CONN_1, P23 CONN_1, P3 CONN_1, P4 CONN_1, P5 CONN_1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

Commit message: initial commit
Other:
- title: 6809PC -> 6502PC
Changed lines of the file:
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@@
 (kicad_sch
-	(version 20231120)
+	(version 20250114)
 	(generator "eeschema")
-	(generator_version "8.0")
+	(generator_version "9.0")
 	(paper "B")
 	(title_block
-		(title "6809PC")
-		(date "2025-06-20")
-		(rev "004")
-		(comment 1 "https://github.com/danwerner21/6809PC")
+		(title "6502PC")
+		(date "2025-10-05")
+		(rev "001")
+		(comment 1 "https://github.com/danwerner21/6502PC")
 		(comment 2 "Based on work by Andrew Lynch and John Coffman")
 	)
+	(text "BYPASS CAPACITORS"
+		(exclude_from_sim no)
+		(at 255.27 168.91 0)
+		(effects
+			(font
+				(size 1.524 1.524)
+			)
+			(justify left bottom)
+		)
+	)
+	(text "MOUNTING HOLES"
+		(exclude_from_sim no)
+		(at 45.72 194.31 0)
+		(effects
+			(font
+				(size 1.524 1.524)
+			)
+			(justify left bottom)
+		)
+	)
+	(text "ATX Connector"
+		(exclude_from_sim no)
+		(at 125.73 125.73 0)
+		(effects
+			(font
+				(size 1.524 1.524)
+			)
+			(justify left bottom)
+		)
+	)
+	(text "ATX Power Supply Control Circuit"
+		(exclude_from_sim no)
+		(at 228.6 85.09 0)
+		(effects
+			(font
+				(size 3.048 3.048)
+			)
+			(justify left bottom)
+		)
+	)
 	(junction
 		(at 226.06 207.01)
@@
 		)
 	)
-	(text "BYPASS CAPACITORS"
-		(exclude_from_sim no)
-		(at 255.27 168.91 0)
-		(effects
-			(font
-				(size 1.524 1.524)
-			)
-			(justify left bottom)
-		)
-	)
-	(text "MOUNTING HOLES"
-		(exclude_from_sim no)
-		(at 45.72 194.31 0)
-		(effects
-			(font
-				(size 1.524 1.524)
-			)
-			(justify left bottom)
-		)
-	)
-	(text "ATX Connector"
-		(exclude_from_sim no)
-		(at 125.73 125.73 0)
-		(effects
-			(font
-				(size 1.524 1.524)
-			)
-			(justify left bottom)
-		)
-	)
-	(text "ATX Power Supply Control Circuit"
-		(exclude_from_sim no)
-		(at 228.6 85.09 0)
-		(effects
-			(font
-				(size 3.048 3.048)
-			)
-			(justify left bottom)
-		)
-	)
 	(label "PWR_ON"
 		(at 323.85 110.49 180)
-		(fields_autoplaced yes)
 		(effects
 			(font
@@
 	(label "VCC"
 		(at 154.94 92.71 0)
-		(fields_autoplaced yes)
 		(effects
 			(font
@@
 	(label "5VSB"
 		(at 213.36 83.82 270)
-		(fields_autoplaced yes)
 		(effects
 			(font
