File: Reset.kicad_sch (KiCad schematic)
At the start: 5 parts, among them SW2 RESET, U17 74LS14, U29 DS1233

Commit message: initial commit
Other:
- title: 6809PC -> 6502PC
Changed lines of the file:
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@@
 (kicad_sch
-	(version 20231120)
+	(version 20250114)
 	(generator "eeschema")
-	(generator_version "8.0")
+	(generator_version "9.0")
 	(paper "A")
 	(title_block
-		(title "6809PC")
-		(date "2025-06-20")
-		(rev "004")
-		(comment 1 "https://github.com/danwerner21/6809PC")
+		(title "6502PC")
+		(date "2025-10-05")
+		(rev "001")
+		(comment 1 "https://github.com/danwerner21/6502PC")
 		(comment 2 "Based on work by Andrew Lynch and John Coffman")
 	)
@@
 	(label "VCC"
 		(at 105.41 78.74 270)
-		(fields_autoplaced yes)
 		(effects
 			(font
@@
 	(label "GND"
 		(at 100.33 78.74 270)
-		(fields_autoplaced yes)
 		(effects
 			(font
