File: Spare.kicad_sch (KiCad schematic)
At the start: 10 parts, among them U10 74LS32, U16 74LS32, U17 74LS14, U18 74LS06, U21 74LS00, U22 74LS74, U4 74LS86, U5 74LS02, U6 74LS00, U9 74LS08

Commit message: initial commit
Parts:
- added U1: 74LS04, Custom:STD_DDW_DIP14, symbol 74xx:74LS04
- added U15: 74LS08, Custom:STD_DDW_DIP14, symbol 74xx:74LS08
- added unit 2 of U17
- added unit 1 of U21
Connections:
- no-connect marks 52 -> 65
Other:
- title: 6809PC -> 6502PC

Commit message: V1.1
Parts:
- added unit 1 of U5
Connections:
- no-connect marks 65 -> 68
Changed lines of the file:
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@@
 	(title_block
 		(title "6502PC")
-		(date "2025-10-05")
-		(rev "001")
+		(date "2025-12-21")
+		(rev "002")
 		(comment 1 "https://github.com/danwerner21/6502PC")
 		(comment 2 "Based on work by Andrew Lynch and John Coffman")
@@
 	)
 	(no_connect
+		(at 213.36 179.07)
+	)
+	(no_connect
 		(at 212.09 160.02)
 	)
@@
 	)
 	(no_connect
+		(at 198.12 181.61)
+	)
+	(no_connect
 		(at 173.99 91.44)
 	)
@@
 	(no_connect
 		(at 220.98 138.43)
+	)
+	(no_connect
+		(at 198.12 176.53)
 	)
 	(no_connect
@@
 				)
 			)
+		)
+	)
+	(symbol
+		(lib_id "74xx:74LS02")
+		(at 205.74 179.07 0)
+		(unit 1)
+		(exclude_from_sim no)
+		(in_bom yes)
+		(on_board yes)
+		(dnp no)
+		(property "Reference" "U5"
+			(at 205.74 177.8 0)
+			(effects
+				(font
+					(size 1.524 1.524)
+				)
+			)
+		)
+		(property "Value" "74LS02"
+			(at 207.01 180.34 0)
+			(effects
+				(font
+					(size 1.524 1.524)
+				)
+			)
+		)
+		(property "Footprint" "Custom:STD_DDW_DIP14"
+			(at 205.74 179.07 0)
+			(effects
+				(font
+					(size 1.27 1.27)
+				)
+				(hide yes)
+			)
+		)
+		(property "Datasheet" "http://www.ti.com/lit/gpn/sn74ls02"
+			(at 205.74 179.07 0)
+			(effects
+				(font
+					(size 1.27 1.27)
+				)
+				(hide yes)
+			)
+		)
+		(property "Description" "quad 2-input NOR gate"
+			(at 205.74 179.07 0)
+			(effects
+				(font
+					(size 1.27 1.27)
+				)
+				(hide yes)
+			)
+		)
+		(pin "7"
+		)
+		(pin "3"
+		)
+		(pin "10"
+		)
+		(pin "9"
+		)
+		(pin "5"
+		)
+		(pin "8"
+		)
+		(pin "11"
+		)
+		(pin "1"
+		)
+		(pin "2"
+		)
+		(pin "4"
+		)
+		(pin "12"
+		)
+		(pin "13"
+		)
+		(pin "14"
+		)
+		(pin "6"
+		)
+		(instances
+			(project "6502PC-6U"
+				(path "/d94f9d60-5ece-4752-b49c-b0d1c95f35bc/00000000-0000-0000-0000-0000526d48aa"
+					(reference "U5")
+					(unit 1)
+				)
+			)
