File: cpu-6502.kicad_sch (KiCad schematic)
At the start: 14 parts, among them P14 16.000Mhz, P15 CPU CLOCK SPEED, U1 74LS04, U13 6502, U17 74LS14, U18 74LS06, U30 74LS163, U31 74LS240, U32 74LS245, U34 74LS244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

Commit message: PCB Routed
Parts:
- U13: footprint Package_DIP:DIP-40_W15.24mm -> Custom:STD_DDW_DIP40
Changed lines of the file:
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@@
 			)
 		)
-		(property "Footprint" "Package_DIP:DIP-40_W15.24mm"
+		(property "Footprint" "Custom:STD_DDW_DIP40"
 			(at 234.95 20.32 0)
 			(effects

Commit message: V1.1
Parts:
- removed U5: 74LS02, Custom:STD_DDW_DIP14, symbol 74xx:74LS02
Connections:
- net GND: now also U34.2 (I0a)
Changed lines of the file:
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@@
 	(title_block
 		(title "6502PC")
-		(date "2025-10-05")
-		(rev "001")
+		(date "2025-12-21")
+		(rev "002")
 		(comment 1 "https://github.com/danwerner21/6502PC")
 		(comment 2 "Based on work by Andrew Lynch and John Coffman")
@@
 	(wire
 		(pts
-			(xy 200.66 185.42) (xy 208.28 185.42)
-		)
-		(stroke
-			(width 0)
-			(type default)
-		)
-	)
-	(wire
-		(pts
 			(xy 50.8 88.9) (xy 66.04 88.9)
 		)
@@
 	(wire
 		(pts
-			(xy 200.66 190.5) (xy 208.28 190.5)
-		)
-		(stroke
-			(width 0)
-			(type default)
-		)
-	)
-	(wire
-		(pts
 			(xy 106.68 73.66) (xy 120.65 73.66)
 		)
@@
 		)
 	)
-	(global_label "CLK"
-		(shape input)
-		(at 200.66 190.5 180)
-		(effects
-			(font
-				(size 1.524 1.524)
-			)
-			(justify right)
-		)
-		(property "Intersheetrefs" "${INTERSHEET_REFS}"
-			(at 200.66 190.5 0)
-			(effects
-				(font
-					(size 1.27 1.27)
-				)
-				(hide yes)
-			)
-		)
-	)
 	(global_label "CPU_R/W"
 		(shape input)
@@
 		)
 	)
-	(global_label "CPU_E"
-		(shape input)
-		(at 200.66 185.42 180)
-		(effects
-			(font
-				(size 1.524 1.524)
-			)
-			(justify right)
-		)
-		(property "Intersheetrefs" "${INTERSHEET_REFS}"
-			(at 200.66 185.42 0)
-			(effects
-				(font
-					(size 1.27 1.27)
-				)
-				(hide yes)
-			)
-		)
-	)
 	(global_label "CPU_D2"
 		(shape bidirectional)
@@
 	)
 	(symbol
-		(lib_id "74xx:74LS02")
-		(at 215.9 187.96 0)
-		(unit 1)
-		(exclude_from_sim no)
-		(in_bom yes)
-		(on_board yes)
-		(dnp no)
-		(property "Reference" "U5"
-			(at 215.9 186.69 0)
-			(effects
-				(font
-					(size 1.524 1.524)
-				)
-			)
-		)
-		(property "Value" "74LS02"
-			(at 217.17 189.23 0)
-			(effects
-				(font
-					(size 1.524 1.524)
-				)
-			)
-		)
-		(property "Footprint" "Custom:STD_DDW_DIP14"
-			(at 215.9 187.96 0)
-			(effects
-				(font
-					(size 1.27 1.27)
-				)
-				(hide yes)
-			)
-		)
-		(property "Datasheet" "http://www.ti.com/lit/gpn/sn74ls02"
-			(at 215.9 187.96 0)
-			(effects
-				(font
-					(size 1.27 1.27)
-				)
-				(hide yes)
-			)
-		)
-		(property "Description" "quad 2-input NOR gate"
-			(at 215.9 187.96 0)
-			(effects
-				(font
-					(size 1.27 1.27)
-				)
-				(hide yes)
-			)
-		)
-		(pin "7"
-		)
-		(pin "3"
-		)
-		(pin "10"
-		)
-		(pin "9"
-		)
-		(pin "5"
-		)
-		(pin "8"
-		)
-		(pin "11"
-		)
-		(pin "1"
-		)
-		(pin "2"
-		)
-		(pin "4"
-		)
-		(pin "12"
-		)
-		(pin "13"
-		)
-		(pin "14"
-		)
-		(pin "6"
-		)
-		(instances
-			(project "6x0x-6U"
-				(path "/d94f9d60-5ece-4752-b49c-b0d1c95f35bc/00000000-0000-0000-0000-0000526c8e8e"
-					(reference "U5")
-					(unit 1)
-				)
-			)
-		)
-	)
-	(symbol
 		(lib_id "power:VCC")
 		(at 394.97 59.69 0)
@@
 					(unit 1)
 				)
+			)
+		)
+	)
+	(symbol
+		(lib_id "power:GND")
+		(at 223.52 187.96 0)
+		(unit 1)
+		(exclude_from_sim no)
+		(in_bom yes)
+		(on_board yes)
+		(dnp no)
+		(property "Reference" "#PWR0182"
+			(at 223.52 187.96 0)
+			(effects
+				(font
+					(size 0.762 0.762)
+				)
+				(hide yes)
+			)
+		)
+		(property "Value" "GND"
+			(at 223.52 189.738 0)
+			(effects
+				(font
+					(size 0.762 0.762)
+				)
+				(hide yes)
+			)
+		)
+		(property "Footprint" ""
+			(at 223.52 187.96 0)
+			(effects
+				(font
+					(size 1.27 1.27)
+				)
+				(hide yes)
+			)
+		)
+		(property "Datasheet" ""
+			(at 223.52 187.96 0)
+			(effects
+				(font
+					(size 1.27 1.27)
+				)
+				(hide yes)
+			)
+		)
+		(property "Description" "Power symbol creates a global label with name \"GND\" , ground"
+			(at 223.52 187.96 0)
+			(effects
+				(font
+					(size 1.27 1.27)
+				)
+				(hide yes)
+			)
+		)
+		(pin "1"
+		)
+		(instances
+			(project "6502PC-6U"
+				(path "/d94f9d60-5ece-4752-b49c-b0d1c95f35bc/00000000-0000-0000-0000-0000526c8e8e"
+					(reference "#PWR0182")
+					(unit 1)
+				)
