File: memory-map.kicad_sch (KiCad schematic)
At the start: 12 parts, among them K1 ROM SELECT, P1 SHADOW ADDR, U1 74LS04, U11 27C256, U17 74LS14, U2 74LS244, U3 74LS682, U4 74LS86, U5 74LS02, U6 74LS00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

Commit message: initial commit
Other:
- title: 6809PC -> 6502PC

Commit message: PCB Routed
Parts:
- U11: footprint Package_DIP:DIP-28_W15.24mm -> Custom:STD_DDW_DIP28
Changed lines of the file:
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@@
 			)
 		)
-		(property "Footprint" "Package_DIP:DIP-28_W15.24mm"
+		(property "Footprint" "Custom:STD_DDW_DIP28"
 			(at 360.68 68.58 0)
 			(effects
